File: Electronique/Carte Robot (base sur un Teensy 3.6)/CarteRobotTeensy/CarteRobot-Teensy.kicad_pcb (KiCad board)
At the start: 2 copper layers, 95.5 x 88.5 mm, 41 parts, among them J1 Conn_Bat2, J10 Conn_01x03, J11 Conn_01x05, J12 Conn_01x05, J13 Conn_01x04, J14 Conn_02x04_Counter_Clockwise, J15 Conn_01x04, J16 Conn_01x04, J17 Conn_01x06, J18 Adaptateur-Servo-Dynamixel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

Commit message: modif elec + modif bom
Parts:
- removed D3, D4: LED, LED_THT:LED_D5.0mm_Clear
- removed J16: Conn_01x04, Connector_Molex:Molex_KK-254_AE-6410-04A_1x04_P2.54mm_Vertical
- removed J17: Conn_01x06, Connector_Molex:Molex_KK-254_AE-6410-06A_1x06_P2.54mm_Vertical
- removed J18: Adaptateur-Servo-Dynamixel, Mes_empreintes:Adaptateur-Servo-Dynamixel
- removed J20, J22: Conn_01x07, Connector_Molex:Molex_KK-254_AE-6410-07A_1x07_P2.54mm_Vertical
- removed J21: Conn_02x04_Counter_Clockwise, Connector_PinHeader_2.54mm:PinHeader_2x04_P2.54mm_Vertical
- removed R4, R5: 500, Resistor_THT:R_Axial_DIN0207_L6.3mm_D2.5mm_P10.16mm_Horizontal
- J15: value Conn_01x04 -> Shield-Actionneurs; footprint Connector_Molex:Molex_KK-254_AE-6410-04A_1x04_P2.54mm_Vertical -> Mes_empreintes:Adaptateur-Servo-Dynamixel; moved to B.Cu
- J19: value Conn_01x04 -> Conn_IHM
- J6: value Conn_01x04 -> Conn_DriverD
- J7: value Conn_01x04 -> Conn_DriverG
- moved J19 22.0 mm to (84.0, 134.0), turned to 0 degrees
- moved J12 20.9 mm to (59.0, 122.1), turned to 90 degrees
- moved J11 14.4 mm to (78.1, 134.0)
- moved J15 11.2 mm to (68.1, 76.0), turned to 270 degrees
- moved J14 8.35 mm to (66.0, 99.6), turned to 180 degrees
- moved J5 3.00 mm to (75.0, 63.0)
- moved J13 2.14 mm to (67.5, 55.0)
Connections:
- J11 pad 3: /CODG_A -> (no net)
- J11 pad 4: /CODG_B -> (no net)
- J13 pad 2: /RX2 -> /TX1
- J13 pad 3: /TX2 -> /RX1
- J14 pad 1: /IRQ -> GND
- J14 pad 2: /MISO1 -> +3V3
- J14 pad 3: /MOSI1 -> /CE
- J14 pad 4: /SCK1 -> /CS0
- J14 pad 5: /CS1 -> /SCK0
- J14 pad 6: /CE -> /MOSI0
- J14 pad 7: +3V3 -> /MISO0
- J14 pad 8: GND -> /IRQ
- J15 pad 1: +3V3 -> /Varu
- J15 pad 2: GND -> /RX3
- J15 pad 4: /RX3 -> GND
- J19 pad 2: /RX5 -> /TX4
- J19 pad 3: /TX5 -> /RX4
- J19 pad 4: +5V -> /Von
- J5 pad 11: /RX2 -> /IRQ
- J5 pad 12: /TX2 -> /CS0
- J5 pad 13: (no net) -> /MOSI0
- J5 pad 14: /CE -> /MISO0
- J5 pad 16: /IRQ -> (no net)
- J5 pad 17: /LED2 -> (no net)
- J5 pad 18: /LED3 -> (no net)
- J5 pad 19: /CODG_A -> /SCK0
- J5 pad 2: /MOSI1 -> /RX1
- J5 pad 20: /CODG_B -> /CODD_B
- J5 pad 21: /CODD_B -> /CODD_A
- J5 pad 22: /CODD_A -> /CE
- J5 pad 23: /CS1 -> /RX4
- J5 pad 24: /SCK1 -> /TX4
- J5 pad 25: /TX5 -> (no net)
- J5 pad 26: /RX5 -> (no net)
- J5 pad 3: /MISO1 -> /TX1
- J5 pad 36: /14 -> (no net)
- J5 pad 37: /15 -> (no net)
- J5 pad 38: /16 -> (no net)
- J5 pad 39: /17 -> (no net)
- J5 pad 42: /20 -> /PWM2
- J5 pad 43: /21 -> /PWM1
- J5 pad 44: /22 -> (no net)
- J5 pad 5: /CAN0TX -> (no net)
- J5 pad 6: /CAN0RX -> (no net)
Routing:
- net +3V3: track 282.3 -> 0.00 mm
- net +5V: track 204.0 -> 0.00 mm
- net /Varu: track 147.8 -> 0.00 mm
- net /MOSI1: track 61.4 -> 0.00 mm
- net /SCK1: track 59.1 -> 0.00 mm
- net /20: track 57.1 -> 0.00 mm
- net /SCL0: track 57.1 -> 0.00 mm
- net /22: track 56.9 -> 0.00 mm
- net /21: track 56.1 -> 0.00 mm
- net /SDA0: track 55.6 -> 0.00 mm
- net /MISO1: track 46.8 -> 0.00 mm
- net /TX2: track 46.6 -> 0.00 mm
- net /RX2: track 44.2 -> 0.00 mm
- net /STEP_G: track 44.1 -> 0.00 mm
- net /DIR_G: track 43.5 -> 0.00 mm
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- removed copper zone on B.Cu, net GND
- removed copper zone on F.Cu, net GND
