File: Electronique/Carte Robot (base sur un Teensy 3.6)/CarteRobotTeensy/CarteRobot-Teensy.sch (KiCad schematic (older format))
At the start: 27 parts, among them J1 Conn_Bat2, J10 Conn_01x03, J11 Conn_01x05, J12 Conn_01x05, J13 Conn_01x04, J14 Conn_02x04_Counter_Clockwise, J15 Conn_01x04, J18 Adaptateur-Servo-Dynamixel, J2 Conn_Bat1, J22 Conn_01x07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

Commit message: Premiere version pcb
Parts:
- added D3, D4: LED, LED_THT:LED_D5.0mm_Clear, symbol Device:LED
- added F1: Fuse, Fuse:Fuse_Littelfuse_372_D8.50mm, symbol Device:Fuse
- added H1, H2, H3, H4: MountingHole, MountingHole:MountingHole_3.2mm_M3_DIN965_Pad, symbol Mechanical:MountingHole
- added J16, J19: Conn_01x04, Connector_Molex:Molex_KK-254_AE-6410-04A_1x04_P2.54mm_Vertical, symbol Connector_Generic:Conn_01x04
- added J17: Conn_01x06, Connector_Molex:Molex_KK-254_AE-6410-06A_1x06_P2.54mm_Vertical, symbol Connector_Generic:Conn_01x06
- added J20: Conn_01x07, Connector_Molex:Molex_KK-254_AE-6410-07A_1x07_P2.54mm_Vertical, symbol Connector_Generic:Conn_01x07
- added J21: Conn_02x04_Counter_Clockwise, Connector_PinHeader_2.54mm:PinHeader_2x04_P2.54mm_Vertical, symbol Connector_Generic:Conn_02x04_Counter_Clockwise
- added R4, R5: 500, Resistor_THT:R_Axial_DIN0207_L6.3mm_D2.5mm_P10.16mm_Horizontal, symbol Device:R
- R1: value 100k -> 500
- R2, R3: footprint (none) -> Resistor_THT:R_Axial_DIN0207_L6.3mm_D2.5mm_P10.16mm_Horizontal
Connections:
- net +3V3: now also J20.7 (Pin_7), J21.7 (Pin_7), J21.8 (Pin_8)
- net +5V: now also J16.3 (Pin_3), J17.1 (Pin_1), J19.4 (Pin_4), J21.1 (Pin_1), J21.2 (Pin_2), J21.3 (Pin_3), J21.4 (Pin_4)
- net 20: now also J20.3 (Pin_3)
- net 21: now also J20.2 (Pin_2)
- net 22: now also J20.1 (Pin_1)
- net A1D: now also J6.3 (Pin_3); no longer J6.2 (Pin_2)
- net DIR_G: now also J5.27 (35); no longer J5.28 (36)
- net GND: now also J18.4, J18.5, D3.1 (K), D4.1 (K), J16.4 (Pin_4), J17.6 (Pin_6), J19.1 (Pin_1), J20.6 (Pin_6), J21.5 (Pin_5), J21.6 (Pin_6)
- net RX3: now also J18.6; no longer J18.3
- net SCL0: now also J20.4 (Pin_4)
- net SDA0: now also J20.5 (Pin_5)
- net STEP_G: now also J5.28 (36); no longer J5.27 (35)
- net TX3: now also J18.7; no longer J18.2
- net LED2: now reaches J5.17 (25)
- net LED2: now also R4.1
- net LED3: now reaches J5.18 (26)
- net LED3: now also R5.1
- net CODG_A: now reaches J5.19 (27)
- net CODG_A: now also J11.3 (Pin_3)
- net CODG_B: now reaches J5.20 (28)
- net CODG_B: now also J11.4 (Pin_4)
- net CODD_B: now reaches J5.21 (29)
- net CODD_B: now also J12.4 (Pin_4)
- net CODD_A: now reaches J5.22 (30)
- net CODD_A: now also J12.3 (Pin_3)
- net TX5: now reaches J5.25 (33)
- net TX5: now also J19.3 (Pin_3)
- net RX5: now reaches J5.26 (34)
- net RX5: now also J19.2 (Pin_2)
- net 14: now reaches J5.36 (14)
- net 14: now also J17.5 (Pin_5)
- net 15: now reaches J5.37 (15)
- net 15: now also J17.4 (Pin_4)
- net 16: now reaches J5.38 (16)
- net 16: now also J17.3 (Pin_3)
- net 17: now reaches J5.39 (17)
- net 17: now also J17.2 (Pin_2)
- net CAN0TX: now reaches J5.5 (3)
- net CAN0TX: now also J16.2 (Pin_2)
- net CAN0RX: now reaches J5.6 (4)
- net CAN0RX: now also J16.1 (Pin_1)
- net at D2.1 (K), J1.1 (Pin_1): now also F1.2; no longer J3.2 (Pin_2)
- net at A1.3 (A2): now also J6.4 (Pin_4); no longer J6.1 (Pin_1)
- net at A1.5 (B1): now also J6.2 (Pin_2); no longer J6.3 (Pin_3)
- net at A1.6 (B2): now also J6.1 (Pin_1); no longer J6.4 (Pin_4)
- new net: F1.1, J3.2 (Pin_2)
- new net: D3.2 (A), R4.2
- new net: D4.2 (A), R5.2
- no-connect marks 0 -> 14
Other:
- moved on the sheet: D2, J14, J15

Commit message: modif elec + modif bom
Parts:
- removed D3, D4: LED, LED_THT:LED_D5.0mm_Clear, symbol Device:LED
- removed J15, J16: Conn_01x04, Connector_Molex:Molex_KK-254_AE-6410-04A_1x04_P2.54mm_Vertical, symbol Connector_Generic:Conn_01x04
- removed J17: Conn_01x06, Connector_Molex:Molex_KK-254_AE-6410-06A_1x06_P2.54mm_Vertical, symbol Connector_Generic:Conn_01x06
- removed J18: Adaptateur-Servo-Dynamixel, Mes_empreintes:Adaptateur-Servo-Dynamixel, symbol Mes_symboles:Adaptateur-Servo-Dynamixel
- removed J20, J22: Conn_01x07, Connector_Molex:Molex_KK-254_AE-6410-07A_1x07_P2.54mm_Vertical, symbol Connector_Generic:Conn_01x07
- removed J21: Conn_02x04_Counter_Clockwise, Connector_PinHeader_2.54mm:PinHeader_2x04_P2.54mm_Vertical, symbol Connector_Generic:Conn_02x04_Counter_Clockwise
- added J15: Shield-Actionneurs, Mes_empreintes:Adaptateur-Servo-Dynamixel, symbol Mes_symboles:Shield-Actionneurs
- added R6, R7, R8, R9: 390k, symbol Device:R
- J14: symbol Connector_Generic:Conn_02x04_Counter_Clockwise -> Connector_Generic:Conn_02x04_Odd_Even
- J19: value Conn_01x04 -> Conn_IHM
- J6: value Conn_01x04 -> Conn_DriverD
- J7: value Conn_01x04 -> Conn_DriverG
- R4, R5: value 500 -> 390k; footprint Resistor_THT:R_Axial_DIN0207_L6.3mm_D2.5mm_P10.16mm_Horizontal -> (none)
Connections:
- net +3V3: now also J14.2 (Pin_2); no longer J14.7 (Pin_7)
- net +5V: now also R8.1, R9.1; no longer J19.4 (Pin_4)
- net CE: now also J14.3 (Pin_3), J5.22 (30); no longer J14.6 (Pin_6), J5.14 (12)
- net CODD_A: now also J5.21 (29); no longer J5.22 (30)
- net CODD_B: now also J5.20 (28); no longer J5.21 (29)
- net CODG_A: now also J5.17 (25), R4.2, R5.1; no longer J11.3 (Pin_3), J5.19 (27)
- net CODG_B: now also J5.18 (26), R6.2, R7.1; no longer J11.4 (Pin_4), J5.20 (28)
- net GND: now also J14.1 (Pin_1), R4.1, J15.4, R6.1; no longer J14.8 (Pin_8)
- net IRQ: now also J14.8 (Pin_8), J5.11 (9); no longer J14.1 (Pin_1), J5.16 (24)
- net RX3: now also J15.2
- net SCL0: now also J15.7
- net SDA0: now also J15.8
- net TX3: now also J15.3
- net Varu: now also J15.1
- net Von: now also J19.4 (Pin_4)
- net MOSI0: now reaches J5.13 (11)
- net MOSI0: now also J14.6 (Pin_6)
- net MS4: now reaches J5.35 (13)
- net at R5.2: now also J11.3 (Pin_3), R8.2
- net 14 renamed MS3
- net 15 renamed MS2
- net 16 renamed MS1
- net 17: no longer names the net of J5.39 (17)
- net 20 renamed PWM2
- net PWM2: now also J15.6
- net 21 renamed PWM1
- net PWM1: now also J15.5
- net 22: no longer names the net of J5.44 (22)
- net CAN0RX renamed SDA2
- net CAN0TX renamed SCL2
- net CS1 renamed RX4
- net RX4: now also J19.3 (Pin_3); no longer J14.5 (Pin_5)
- removed net LED2: J5.17 (25), R4.1
- removed net LED3: J5.18 (26), R5.1
- net MISO1 renamed TX1
- net TX1: now also J13.2 (Pin_2); no longer J14.2 (Pin_2)
- net MOSI1 renamed RX1
- net RX1: now also J13.3 (Pin_3); no longer J14.3 (Pin_3)
- removed net RX2: J13.2 (Pin_2), J5.11 (9)
- net RX5: no longer names the net of J5.26 (34)
- net RX5: no longer J19.2 (Pin_2)
- net SCK1 renamed CS0
- net CS0: now also J5.12 (10); no longer J5.24 (32)
- removed net TX2: J13.3 (Pin_3), J5.12 (10)
- net TX5: no longer names the net of J5.25 (33)
- net TX5: no longer J19.3 (Pin_3)
- new net: J11.4 (Pin_4), R7.2, R9.2
- new net MISO0: J14.7 (Pin_7), J5.14 (12)
- new net SCK0: J14.5 (Pin_5), J5.19 (27)
- new net TX4: J19.2 (Pin_2), J5.24 (32)
- no-connect marks 14 -> 12
Other:
- moved on the sheet: A1, A2, C1, C2, D1, D2, F1, H1, H2, H3, H4, J1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
